Commit message: wheelを地面においてある状態とlimbについてある状態に変更可能になった。ただし、交代のたびに初期姿勢に戻るのでそれの対処が必要

File: xacro/palette.xacro (robot description, xacro)
@@ -5,5 +5,6 @@
    <xacro:include filename="$(find urdf_tutorial)/xacro/palette_body.xacro" />
    <!-- 追加: ホイール有無の引数（デフォルト: あり） -->
-   <xacro:arg name="use_wheel" default="true"/>
+   <!-- <xacro:arg name="use_wheel" default="true"/> -->
+   <xacro:arg name="attach_wheel" default="true"/>
    <link name="palette_link">
     </link>
@@ -90,6 +91,19 @@
     <xacro:limb name="limb_n_14" base_frame="palette_link_4" p="${0*pi/180}" y="${0*pi/180}" r="${0*pi/180}" />
     <!-- <xacro:limb name="limb_n_15" base_frame="palette_link_3" p="${0*pi/180}" y="${0*pi/180}" r="${0*pi/180}" /> -->
-    <xacro:wheel_d250 name="wheel_n_1" base_frame="palette_link_10" p="${0*pi/180}" y="${90*pi/180}" r="${90*pi/180}" />
+    <!-- <xacro:wheel_d250 name="wheel_n_1" base_frame="palette_link_10" p="${0*pi/180}" y="${90*pi/180}" r="${90*pi/180}" /> -->
     <xacro:palette_body name="body_n_2" base_frame="palette_link_12" p="${0*pi/180}" y="${90*pi/180}" r="${0*pi/180}" />
+    <!-- すでに定義済み: <xacro:arg name="attach_wheel" default="true"/> -->
+    <xacro:if value="$(arg attach_wheel)">
+        <xacro:wheel_d250 name="wheel_n_1"
+                            base_frame="body_n_2_limb_n_2_limb_end_effector"
+                            x="0.034" y_pos="-0.09" z="0.03"
+                            r="${90*pi/180}" p="${0*pi/180}" y="${90*pi/180}"/>
+    </xacro:if>
+    <xacro:unless value="$(arg attach_wheel)">
+        <xacro:wheel_d250 name="wheel_n_1"
+                            base_frame="palette_link_10"
+                            x="0.0" y_pos="0.0" z="0.0"
+                            r="${90*pi/180}" p="${0*pi/180}" y="${90*pi/180}"/>
+    </xacro:unless>
     <!-- <xacro:limb name="palette_body_n_2" base_frame="palette_body_n_2_link_2" p="0" y="${0*pi/180}" r="${0*pi/180}" /> -->
     <!-- <xacro:if value="$(arg use_wheel)">

File: xacro/wheel_d250_with_connector.xacro (robot description, xacro)
@@ -1,21 +1,30 @@
 <?xml version="1.0"?>
 <robot xmlns:xacro="http://www.ros.org/wiki/xacro" name="wheel_d250_robot">
-    <!-- Define a macro for the wheel -->
-    <xacro:macro name="wheel_d250" params="name base_frame r p y" >
-        <!-- Base link -->
-        <joint name="${name}_joint" type="fixed">
-            <parent link="${base_frame}"/>
-            <child link="${name}_base_wheel_link"/>
-            <origin xyz="0 0 0" rpy="${r} ${p} ${y}"/>
-        </joint>
-        <link name="${name}_base_wheel_link">
-            <visual>
-            <origin xyz="0 0 0" rpy="${pi/2} ${pi} 0" />
-                <geometry>
-                    <mesh filename="package://urdf_tutorial/stl/wheel_d250_with_connector.stl" scale="0.001 0.001 0.001"/>
-                </geometry>
-                <material name="silver"/>
-            </visual>
-        </link>
-    </xacro:macro>
+  <!--
+    wheel_d250 マクロ
+    - name: このホイールの識別名
+    - base_frame: 接続元リンク名
+    - r,p,y: 回転角 (ラジアン)
+    - x,y_pos,z: 親リンクからの位置 (m)
+  -->
+  <xacro:macro name="wheel_d250" params="name base_frame r p y x:=0.0 y_pos:=0.0 z:=0.0">
+    <!-- 親リンクとの固定ジョイント -->
+    <joint name="${name}_joint" type="fixed">
+      <parent link="${base_frame}"/>
+      <child link="${name}_base_wheel_link"/>
+      <!-- ★ 位置と姿勢 -->
+      <origin xyz="${x} ${y_pos} ${z}" rpy="${r} ${p} ${y}"/>
+    </joint>
+    <!-- ベースリンク -->
+    <link name="${name}_base_wheel_link">
+      <visual>
+        <origin xyz="0 0 0" rpy="${pi/2} ${pi} 0"/>
+        <geometry>
+          <mesh filename="package://urdf_tutorial/stl/wheel_d250_with_connector.stl"
+                scale="0.001 0.001 0.001"/>
+        </geometry>
+        <material name="silver"/>
+      </visual>
+    </link>
+  </xacro:macro>
 </robot>

Commit message: limbをゴールまで動かすことと結合ができるようになった

File: xacro/palette.xacro (robot description, xacro)
@@ -4,7 +4,9 @@
    <xacro:include filename="$(find urdf_tutorial)/xacro/wheel_d250_with_connector.xacro" />
    <xacro:include filename="$(find urdf_tutorial)/xacro/palette_body.xacro" />
+   <xacro:include filename="$(find urdf_tutorial)/xacro/gripper.xacro" />
    <!-- 追加: ホイール有無の引数（デフォルト: あり） -->
    <!-- <xacro:arg name="use_wheel" default="true"/> -->
-   <xacro:arg name="attach_wheel" default="true"/>
+   <xacro:arg name="attach_wheel" default="false"/>
+   <xacro:arg name="attach_gripper" default="false"/>
    <link name="palette_link">
     </link>
@@ -22,4 +24,6 @@
     <link name="palette_link_12"/>
     <link name="palette_link_13"/>
+    <link name="palette_link_14"/>
+    <link name="palette_link_15"/>
     <joint name="palette_joint_1" type="fixed">
         <parent link="palette_link"/>
@@ -40,10 +44,10 @@
         <parent link="palette_link"/>
         <child link="palette_link_4"/>
-        <origin xyz="0 -0.28 0" rpy="0 0 0"/>
+        <origin xyz="0.20 -0.78 0" rpy="0 0 0"/>
     </joint>
     <joint name="palette_joint_5" type="fixed">
         <parent link="palette_link"/>
         <child link="palette_link_5"/>
-        <origin xyz="0.28 -0.28 0" rpy="0 0 0"/>
+        <origin xyz="0.48 -0.78 0" rpy="0 0 0"/>
     </joint>
     <joint name="palette_joint_6" type="fixed">
@@ -87,7 +91,30 @@
         <origin xyz="1.12 -1.36 0" rpy="0 0 0"/>
     </joint>
-    <xacro:limb name="limb_n_12" base_frame="palette_link_7" p="${0*pi/180}" y="${0*pi/180}" r="${0*pi/180}" />
-    <xacro:limb name="limb_n_13" base_frame="palette_link_5" p="${0*pi/180}" y="${0*pi/180}" r="${0*pi/180}" />
-    <xacro:limb name="limb_n_14" base_frame="palette_link_4" p="${0*pi/180}" y="${0*pi/180}" r="${0*pi/180}" />
+    <joint name="palette_joint_14" type="fixed">
+        <parent link="palette_link"/>
+        <child link="palette_link_14"/>
+        <origin xyz="1.03 -0.50 0.0" rpy="0 0 0"/>
+    </joint>
+    <joint name="palette_joint_15" type="fixed">
+        <parent link="palette_link"/>
+        <child link="palette_link_15"/>
+        <origin xyz="1.3 -0.50 0.0" rpy="0 0 0"/>
+    </joint>
+    <xacro:limb name="limb_n_12" base_frame="palette_link_5" p="${0*pi/180}" y="${0*pi/180}" r="${0*pi/180}" />
+    <xacro:limb name="limb_n_13" base_frame="palette_link_14" p="${0*pi/180}" y="${0*pi/180}" r="${0*pi/180}" />
+    <xacro:limb name="limb_n_14" base_frame="palette_link_15" p="${0*pi/180}" y="${0*pi/180}" r="${0*pi/180}" />
+    <xacro:if value="$(arg attach_gripper)">
+        <xacro:gripper name="gripper_n_1"
+                            base_frame="limb_n_12_limb_end_effector"
+                            x="0.0" y_pos="0.0" z="0.0"
+                            r="${-90*pi/180}" p="${0*pi/180}" y="${90*pi/180}"/>
+    </xacro:if>
+    <xacro:unless value="$(arg attach_gripper)">
+        <xacro:gripper name="gripper_n_1"
+                            base_frame="palette_link_4"
+                            x="0.0" y_pos="0.0" z="0.0"
+                            r="${90*pi/180}" p="${0*pi/180}" y="${90*pi/180}"/>
+    </xacro:unless>
+    <!-- <xacro:gripper name="gripper_n_1" base_frame="palette_link_4" x="0.0" y_pos="0.0" z="0.0" p="${0*pi/180}" y="${90*pi/180}" r="${90*pi/180}" /> -->
     <!-- <xacro:limb name="limb_n_15" base_frame="palette_link_3" p="${0*pi/180}" y="${0*pi/180}" r="${0*pi/180}" /> -->
     <!-- <xacro:wheel_d250 name="wheel_n_1" base_frame="palette_link_10" p="${0*pi/180}" y="${90*pi/180}" r="${90*pi/180}" /> -->
